Commit message: Fix stls in urdf model

File: bullet/TEO.urdf (robot description, URDF)
Before this commit: robot teo, 31 links, 30 joints
Joints:
- joint l_ankle_pitch: limit lower=-0.314159265359 upper=0.349065850399 effort=85.0 velocity=4.0 -> lower=-0.4031710572 upper=0.44331363 effort=85.0 velocity=4.0
- joint l_ankle_roll: axis -1 0 0 -> 1 0 0; limit lower=-0.436332312999 upper=0.436332312999 effort=65.0 velocity=4.0 -> lower=-0.7417649321 upper=0.3473205211 effort=65.0 velocity=4.0
- joint l_hip_pitch: limit lower=-0.523598775598 upper=0.785398163397 effort=60.0 velocity=4.0 -> lower=-0.5515240436 upper=0.7382742736 effort=60.0 velocity=4.0
- joint l_hip_roll: axis -1 0 0 -> 1 0 0; limit lower=-0.349065850399 upper=0.349065850399 effort=65.0 velocity=4.0 -> lower=-0.2181661565 upper=0.2478367538 effort=65.0 velocity=4.0
- joint l_hip_yaw: axis 0 0 1.0 -> 0 0 1; limit lower=-1.57079632679 upper=1.57079632679 effort=45.0 velocity=4.0 -> lower=-0.4869468613 upper=0.5724679947 effort=45.0 velocity=4.0
- joint l_knee_pitch: limit lower=-0.0872664625997 upper=1.3962634016 effort=140.0 velocity=4.0 -> lower=-1.0698868315 upper=1.4381513036 effort=140.0 velocity=4.0
- joint l_shoulder_yaw: axis 0 0 -1 -> 0 0 1
- joint l_sole_joint: origin xyz=0 0 -0.124 rpy=0 0 0 -> xyz=0 0 -0.123005 rpy=0 0 0
- joint l_wrist_yaw: axis 0 0 -1 -> 0 0 1
- joint r_ankle_pitch: limit lower=-0.314159265359 upper=0.349065850399 effort=85.0 velocity=4.0 -> lower=-0.4031710572 upper=0.44331363 effort=85.0 velocity=4.0
- joint r_ankle_roll: axis -1 0 0 -> 1 0 0; limit lower=-0.436332312999 upper=0.436332312999 effort=65.0 velocity=4.0 -> lower=-0.3473205211 upper=0.7417649321 effort=65.0 velocity=4.0
- joint r_hip_pitch: limit lower=-0.523598775598 upper=0.785398163397 effort=60.0 velocity=4.0 -> lower=-0.5515240436 upper=0.7382742736 effort=60.0 velocity=4.0
- joint r_hip_roll: axis -1 0 0 -> 1 0 0; limit lower=-0.349065850399 upper=0.349065850399 effort=65.0 velocity=4.0 -> lower=-0.2478367538 upper=0.2181661565 effort=65.0 velocity=4.0
- joint r_hip_yaw: axis 0 0 -1.0 -> 0 0 1; limit lower=-1.57079632679 upper=1.57079632679 effort=45.0 velocity=4.0 -> lower=-0.5724679947 upper=0.4869468613 effort=45.0 velocity=4.0
- joint r_knee_pitch: limit lower=-0.0872664625997 upper=1.3962634016 effort=140.0 velocity=4.0 -> lower=-1.0698868315 upper=1.4381513036 effort=140.0 velocity=4.0
- joint r_shoulder_pitch: axis 0 -1.0 0 -> 0 1 0
- joint r_shoulder_yaw: axis 0 0 -1 -> 0 0 1
- joint r_sole_joint: origin xyz=0 0 -0.124 rpy=0 0 0 -> xyz=0 0 -0.123005 rpy=0 0 0
- joint r_wrist_pitch: axis 0 -1.0 0 -> 0 1 0
- joint waist_pitch: limit lower=-0.174532925199 upper=0.174532925199 effort=30.0 velocity=3.0 -> lower=-1.5777776438 upper=0.1762782545 effort=30.0 velocity=3.0
- joint waist_yaw: limit lower=-0.785398163397 upper=0.785398163397 effort=30.0 velocity=3.0 -> lower=-1.0349802464 upper=0.8080874437 effort=30.0 velocity=3.0
